Commit message: urdf finished, now I have to improve it using xacros and adding gazebo stuff

File: src/canyonero_description/urdf/canyonero.urdf (robot description, URDF)
Before this commit: robot cambot, 7 links, 6 joints
Links:
- added link imu_link, mass 0.0458425; visual mesh filename=package://canyonero_description/meshes/9dof_razor_imu.stl
- link kinect_link: mass None -> 0.0458425; geometry visual mesh filename=package://canyonero_description/meshes/kinect.stl
Joints:
- added joint base_link_to_imu: type fixed, parent base_link, child imu_link, origin xyz=1.885 0 1.08 rpy=0 0 -1.57
- joint base_footprint_joint: origin xyz=0 0 2.04 rpy=0 0 0 -> xyz=0 0 1.67 rpy=0 0 0
- joint base_link_to_kinect: origin xyz=2.62 0 0.95 rpy=0 0 0 -> xyz=2.62 0 1.41 rpy=0 0 0
- joint base_to_back_left_wheel: origin xyz=-1.62 1.65 -1.05 rpy=-1.57 0 0 -> xyz=-1.62 1.65 -0.68 rpy=-1.57 0 0
- joint base_to_back_right_wheel: origin xyz=-1.62 -1.65 -1.05 rpy=1.57 0 0 -> xyz=-1.62 -1.65 -0.68 rpy=1.57 0 0
- joint base_to_frontal_left_wheel: origin xyz=1.62 1.65 -1.05 rpy=-1.57 0 0 -> xyz=1.62 1.65 -0.68 rpy=-1.57 0 0
- joint base_to_frontal_right_wheel: origin xyz=1.62 -1.65 -1.05 rpy=1.57 0 0 -> xyz=1.62 -1.65 -0.68 rpy=1.57 0 0

Commit message: adding gazebo stuff

File: src/canyonero_description/urdf/canyonero.urdf (robot description, URDF)
Before this commit: robot cambot, 8 links, 7 joints
Links:
- link back_left_wheel_link: mass 15.23 -> 1.419; geometry collision mesh filename=package://canyonero_description/meshes/canyonero_wheel_coll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; visual mesh filename=package://canyonero_description/meshes/canyonero_wheel.stl
- link back_right_wheel_link: mass 15.23 -> 1.419; geometry collision mesh filename=package://canyonero_description/meshes/canyonero_wheel_coll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; visual mesh filename=package://canyonero_description/meshes/canyonero_wheel.stl
- link base_link: geometry collision mesh filename=package://canyonero_description/meshes/canyonero_plates_col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; visual mesh filename=package://canyonero_description/meshes/canyonero_plates.stl
- link frontal_left_wheel_link: mass 15.23 -> 1.419; geometry collision mesh filename=package://canyonero_description/meshes/canyonero_wheel_coll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; visual mesh filename=package://canyonero_description/meshes/canyonero_wheel.stl
- link frontal_right_wheel_link: mass 15.23 -> 1.419; geometry collision mesh filename=package://canyonero_description/meshes/canyonero_wheel_coll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; visual mesh filename=package://canyonero_description/meshes/canyonero_wheel.stl
- link imu_link: mass 0.0458425 -> 0.01
- link kinect_link: mass 0.0458425 -> 0.564; geometry collision box size=0.07271 0.27794 0.073; visual mesh filename=package://canyonero_description/meshes/kinect.stl

File: src/canyonero_description/urdf/canyonero_base.urdf.xacro (robot description, xacro)
@@ -6,5 +6,6 @@
 -->
 <robot xmlns:xacro="http://ros.org/wiki/xacro">
-	<xacro:include filename="$(find canyonero_description)/urdf/canyonero_wheel.urdf.xacro"/>
+	<xacro:include filename="$(find canyonero_description)/urdf/wheels/canyonero_wheel.urdf.xacro"/>
+	<!--xacro:include filename="$(find canyonero_description)/urdf/wheels/canyonero_wheel.transmission.xacro"/-->
 	<xacro:macro name= "base" params = "name">
 	<!-- BASE-FOOTPRINT -->
@@ -26,10 +27,10 @@
 				<material name = "Red"/>
 			</visual>
-			<!--collision>
+			<collision>
 	      		<origin xyz = "0 0 0" rpy = "0 0 0"/>
 	      		<geometry>
 	        		<mesh filename = "package://canyonero_description/meshes/canyonero_plates_collision.stl"/>
 	      		</geometry>
-	    	</collision-->
+	    	</collision>
 			<inertial>
 	      		<origin rpy = "0 0 0" xyz = "174.84e-3 117.51e-3 -218.86e-3"/>
@@ -43,4 +44,7 @@
 	               		 izz="0.016834"/>
 	    	</inertial>
+	    	<gazebo reference="${name}_link">
+      			<material>Gazebo/Red</material>
+    		</gazebo>
 		</link>
 		<!-- Wheels -->

File: src/canyonero_description/urdf/sensors/canyonero_imu.urdf.xacro (robot description, xacro)
@@ -48,4 +48,5 @@
         </imu>
       </sensor>
+      <material>Gazebo/Red</material>
     </gazebo>
   </xacro:macro>

File: src/canyonero_description/urdf/sensors/canyonero_kinect.urdf.xacro (robot description, xacro)
@@ -34,4 +34,7 @@
                  izz="0.003879257" />
       </inertial>
+      <gazebo reference="camera_link">
+        <material>Gazebo/Black</material>
+      </gazebo>
     </link>
     <!-- RGB camera -->

File: src/canyonero_description/urdf/wheels/canyonero_wheel.urdf.xacro (robot description, xacro)
@@ -15,20 +15,17 @@
 	        	<material name = "Black"/>
 	      	</visual>
-		    <inertial>
-		    	<origin xyz="0.1026 0.0 0.0" rpy="0 0 0"/>
-		        <mass value="1.419"/>
-		        <inertia ixx="0.0165" ixy="0.0" ixz="0.0"
-		                 iyy="0.0106" iyz="0.0"
-		                 izz="0.0106"/>
-		    </inertial>
-	      	<collision>
+		    <!--inertial>
+		    	<origin xyz="1.62*${positionX} 1.65*${positionY} -0.68" rpy="1.57*${reflect} 0 0"/>
+		        <mass value="1.82362"/>
+		        <inertia ixx="0.00499743171" ixy="${ 0.00000004464 * reflect}" ixz="-0.00000002245"
+		                 iyy="0.00499741733" iyz="${-0.00000000164 * reflect}"
+		                 izz="0.00839239692"/>
+		    </inertial-->
+	      	<!--collision>
 	        	<origin xyz="0 0 0" rpy="0 0 0"/>
 	        	<geometry>
-	          		<mesh filename = "package://canyonero_description/meshes/canyonero_wheel_collision.stl"/>
+	          		<mesh filename = "package://canyonero_description/meshes/canyonero_wheel.stl"/>
 	        	</geometry>
-	      	</collision>
-	      	<gazebo reference="${sideY}_${sideX}_wheel_link">
-      			<material>Gazebo/Black</material>
-    		</gazebo>
+	      	</collision-->
 	    </link>
 	    <joint name="${sideY}_${sideX}_wheel_joint" type="continuous">
