Commit message: updating canyonero_description

File: src/canyonero_description/urdf/canyonero_base.urdf.xacro (robot description, xacro)
@@ -7,5 +7,4 @@
 <robot xmlns:xacro="http://ros.org/wiki/xacro">
 	<xacro:include filename="$(find canyonero_description)/urdf/wheels/canyonero_wheel.urdf.xacro"/>
-	<!--xacro:include filename="$(find canyonero_description)/urdf/wheels/canyonero_wheel.transmission.xacro"/-->
 	<xacro:macro name= "base" params = "name">
 	<!-- BASE-FOOTPRINT -->
@@ -34,16 +33,12 @@
 	    	</collision>
 			<inertial>
-	      		<origin rpy = "0 0 0" xyz = "174.84e-3 117.51e-3 -218.86e-3"/>
-	      		<mass value = "15.23"/>
-	      		<!-- inertia at cm or origin?-->
-	      		<inertia ixx = "0.016258"
-	               		 ixy = "0.000432"
-	               		 ixz="-0.000049"
-	               		 iyy="0.019275"
-	               		 iyz="0.000048"
-	               		 izz="0.016834"/>
+	      		<origin xyz="0.023661 -0.000069 -0.036285" rpy="0 0 0" />
+	      		<mass value = "10"/>
+	      		<inertia ixx="0.5284" ixy="-0.0003498" ixz="0.001138"
+	               		 iyy="0.5262" iyz="0.02108"
+	               		 izz="0.9556"/>
 	    	</inertial>
-	    	<gazebo reference="${name}_link">
-      			<material>Gazebo/Red</material>
+				<gazebo reference="${name}_link">
+      		<material>Gazebo/Red</material>
     		</gazebo>
 		</link>
@@ -53,4 +48,9 @@
 	    <xacro:wheel sideX = "back" sideY = "left" positionX = "-1.0" positionY = "1.0" reflect = "-1.0" parent = "${name}"/>
 	    <xacro:wheel sideX = "back" sideY = "right" positionX = "-1.0" positionY = "-1.0" reflect = "1.0" parent = "${name}"/>
+			<gazebo>
+				<plugin name="gazebo_ros_control" filename="libgazebo_ros_control.so">
+				<robotNamespace>canyonero</robotNamespace>
+				</plugin>
+			</gazebo>
 	</xacro:macro>
 </robot>

File: src/canyonero_description/urdf/canyonero_properties.urdf.xacro (robot description, xacro)
@@ -19,30 +19,30 @@
 	<!-- base properties -->
 	<!-- robot's elevation from the ground -->
-	<property name = "rob_pos_Z"	value = "1.67"/>
+	<property name = "rob_pos_Z"	value = "0.167"/>
 	<!-- wheel properties -->
-	<property name = "wheel_pos_X"      value = "1.62"/>
-	<property name = "wheel_pos_Y"      value = "1.65"/>
-	<property name = "wheel_pos_Z"			value = "0.68"/>
+	<property name = "wheel_pos_X"      value = "0.162"/>
+	<property name = "wheel_pos_Y"      value = "0.165"/>
+	<property name = "wheel_pos_Z"			value = "0.068"/>
 	<!-- kinect properties -->
 	<!-- kinect position at the robot -->
-	<xacro:property name="cam_pos_X" value="2.62" />
-	<xacro:property name="cam_pos_Y" value="0" />
-	<xacro:property name="cam_pos_Z" value="1.41" />
+	<xacro:property name="cam_pos_X" value="0.262" />
+	<xacro:property name="cam_pos_Y" value="0.0" />
+	<xacro:property name="cam_pos_Z" value="0.141" />
 	<xacro:property name="cam_or_R" value="${PI / 2}" />
-	<xacro:property name="cam_or_P" value="0" />
+	<xacro:property name="cam_or_P" value="0.0" />
 	<xacro:property name="cam_or_Y" value="${PI / 2}" />
 	<!-- kinect cam position at the kinect itself -->
-	<xacro:property name="cam_px" value="0.29" />
-	<xacro:property name="cam_py" value="-0.1" />
-	<xacro:property name="cam_pz" value="0.19" />
-	<xacro:property name="cam_or" value="0" />
-	<xacro:property name="cam_op" value="0" />
-	<xacro:property name="cam_oy" value="0" />
-	<!-- kinect properties -->
-	<xacro:property name="imu_pos_X" value="1.885"/>
-	<xacro:property name="imu_pos_Y" value="0"/>
-	<xacro:property name="imu_pos_Z" value="1.08"/>
-	<xacro:property name="imu_or_R"	value="0"/>
-	<xacro:property name="imu_or_P" value="0"/>
+	<xacro:property name="cam_px" value="0.029" />
+	<xacro:property name="cam_py" value="-0.01" />
+	<xacro:property name="cam_pz" value="0.019" />
+	<xacro:property name="cam_or" value="0.0" />
+	<xacro:property name="cam_op" value="0.0" />
+	<xacro:property name="cam_oy" value="0.0" />
+	<!-- imu properties -->
+	<xacro:property name="imu_pos_X" value="0.1885"/>
+	<xacro:property name="imu_pos_Y" value="0.0"/>
+	<xacro:property name="imu_pos_Z" value="0.108"/>
+	<xacro:property name="imu_or_R" value="0.0"/>
+	<xacro:property name="imu_or_P" value="0.0"/>
 	<xacro:property name="imu_or_Y" value="${-PI / 2}"/>
 </robot>

File: src/canyonero_description/urdf/sensors/canyonero_imu.urdf.xacro (robot description, xacro)
@@ -16,5 +16,5 @@
         <origin xyz = "0 0 0" rpy = "0 0 0" />
         <geometry>
-          <mesh filename = "package://canyonero_description/meshes/9dof_razor_imu.stl"/>
+          <mesh filename = "package://canyonero_description/meshes/9dof_razor_imu.stl" scale="0.1 0.1 0.1"/>
         </geometry>
         <material name = "Red"/>
@@ -23,5 +23,5 @@
         <mass value="0.01"/>
         <origin xyz="0 0 0"/>
-        <inertia ixx="0.000001" ixy="0" ixz="0" iyy="0.000001" iyz="0" izz="0.000001"/>
+        <inertia ixx="0.0000001" ixy="0.0" ixz="0.0" iyy="0.0000001" iyz="0.0" izz="0.0000001"/>
       </inertial>
     </link>

File: src/canyonero_description/urdf/sensors/canyonero_kinect.urdf.xacro (robot description, xacro)
@@ -17,5 +17,5 @@
        <origin xyz="0 0 0" rpy="${cam_or_R} ${cam_or_P} ${cam_or_Y}"/>
         <geometry>
-         <mesh filename="package://canyonero_description/meshes/kinect.stl"/>
+         <mesh filename="package://canyonero_description/meshes/kinect.stl" scale="0.1 0.1 0.1"/>
         </geometry>
         <material name="DarkGrey" />

File: src/canyonero_description/urdf/wheels/canyonero_wheel.urdf.xacro (robot description, xacro)
@@ -15,17 +15,20 @@
 	        	<material name = "Black"/>
 	      	</visual>
-		    <!--inertial>
-		    	<origin xyz="1.62*${positionX} 1.65*${positionY} -0.68" rpy="1.57*${reflect} 0 0"/>
-		        <mass value="1.82362"/>
-		        <inertia ixx="0.00499743171" ixy="${ 0.00000004464 * reflect}" ixz="-0.00000002245"
-		                 iyy="0.00499741733" iyz="${-0.00000000164 * reflect}"
-		                 izz="0.00839239692"/>
-		    </inertial-->
-	      	<!--collision>
-	        	<origin xyz="0 0 0" rpy="0 0 0"/>
+		    <inertial>
+		    	<origin xyz="0.0 0.0 0.102638" rpy="0 0 0"/>
+		        <mass value="1.419"/>
+		        <inertia ixx="0.01101" ixy="0.0000238" ixz="0.00000223198"
+				        		 iyy="0.01104" iyz="${-0.00000012456 * reflect}"
+				             izz="0.003326"/>
+		    </inertial>
+	      	<collision>
+	        	<origin xyz="0 0 0" rpy="0 ${-PI / 2} 0"/>
 	        	<geometry>
-	          		<mesh filename = "package://canyonero_description/meshes/canyonero_wheel.stl"/>
+	          		<mesh filename = "package://canyonero_description/meshes/canyonero_wheel_collision.stl"/>
 	        	</geometry>
-	      	</collision-->
+	      	</collision>
+	      	<gazebo reference="${sideY}_${sideX}_wheel_link">
+      			<material>Gazebo/Black</material>
+    		</gazebo>
 	    </link>
 	    <joint name="${sideY}_${sideX}_wheel_joint" type="continuous">
@@ -35,4 +38,14 @@
 	      	<axis xyz="0 0 1"/>
 	    </joint>
+			<transmission name="simple_trans">
+			  <type>transmission_interface/SimpleTransmission</type>
+			  <joint name="${sideY}_${sideX}_wheel_joint">
+					<hardwareInterface>EffortJointInterface</hardwareInterface>
+			  </joint>
+			  <actuator name="DC_motor">
+					<mechanicalReduction>1</mechanicalReduction>
+					<hardwareInterface>EffortJointInterface</hardwareInterface>
+			  </actuator>
+			</transmission>
   	</xacro:macro>
 </robot>
