Commit message: Canyonero_gazebo working with all the plugins (roscontrol, kinect and imu). Juampe, we should test the roscontrol part

File: src/canyonero_description/urdf/canyonero.urdf.xacro (robot description, xacro)
@@ -10,12 +10,12 @@
 		<xacro:include filename="$(find canyonero_description)/urdf/sensors/canyonero_kinect.urdf.xacro"/>
 		<xacro:include filename="$(find canyonero_description)/urdf/sensors/canyonero_imu.urdf.xacro"/>
-		<xacro:include filename="$(find canyonero_gazebo)/urdf/canyonero_gazebo.urdf.xacro"/>
-			<!-- Base -->
-			<xacro:wheeled_base name="base"/>
-			<!-- 3D sensor -->
-			<xacro:sensor_kinect parent="base_link"/>
-			<!-- IMU -->
-			<xacro:imu_sensor parent="base_link"/>
-			<!-- Gazebo -->
-			<xacro:canyonero_robot_gazebo/>
+		<xacro:include filename="$(find canyonero_gazebo)/urdf/canyonero.gazebo.xacro"/>
+		<!-- Base -->
+		<xacro:wheeled_base name="base"/>
+		<!-- 3D sensor -->
+		<xacro:sensor_kinect parent="base_link"/>
+		<!-- IMU -->
+		<xacro:imu_sensor parent="base_link"/>
+		<!-- Gazebo -->
+		<xacro:canyonero_robot_gazebo/>
 </robot>

File: src/canyonero_description/urdf/canyonero_base.urdf.xacro (robot description, xacro)
@@ -41,5 +41,5 @@
 		</link>
 		<gazebo reference="${name}_link">
-      <material>Gazebo/Red</material>
+      <material value="Gazebo/Red"/>
     </gazebo>
 		<!-- Wheels -->

File: src/canyonero_description/urdf/canyonero_properties.urdf.xacro (robot description, xacro)
@@ -19,33 +19,33 @@
 	<!-- base properties -->
 	<!-- robot's elevation from the ground -->
-	<property name="rob_pos_Z" value="0.167"/>
+	<xacro:property name="rob_pos_Z" value="0.167"/>
 	<!-- wheel properties -->
-	<property name="wheel_pos_X" value="0.162"/>
-	<property name="wheel_pos_Y" value="0.165"/>
-	<property name="wheel_pos_Z" value="0.068"/>
-	<property name="wheel_torque" value="1.0"/>
-	<property name="wheel_velocity" value="1.0"/>
-	<property name="wheel_radius" value="0.20"/>
+	<xacro:property name="wheel_pos_X" value="0.162"/>
+	<xacro:property name="wheel_pos_Y" value="0.165"/>
+	<xacro:property name="wheel_pos_Z" value="0.068"/>
+	<xacro:property name="wheel_torque" value="1.0"/>
+	<xacro:property name="wheel_velocity" value="1.0"/>
+	<xacro:property name="wheel_radius" value="0.20"/>
 	<!-- kinect properties -->
 	<!-- kinect position at the robot -->
-	<property name="cam_pos_X" value="0.262" />
-	<property name="cam_pos_Y" value="0.0" />
-	<property name="cam_pos_Z" value="0.141" />
-	<property name="cam_or_R" value="${PI / 2}" />
-	<property name="cam_or_P" value="0.0" />
-	<property name="cam_or_Y" value="${PI / 2}" />
+	<xacro:property name="cam_pos_X" value="0.262" />
+	<xacro:property name="cam_pos_Y" value="0.0" />
+	<xacro:property name="cam_pos_Z" value="0.141" />
+	<xacro:property name="cam_or_R" value="${PI / 2}" />
+	<xacro:property name="cam_or_P" value="0.0" />
+	<xacro:property name="cam_or_Y" value="${PI / 2}" />
 	<!-- kinect cam position at the kinect itself -->
-	<property name="cam_px" value="0.029" />
-	<property name="cam_py" value="-0.01" />
-	<property name="cam_pz" value="0.019" />
-	<property name="cam_or" value="0.0" />
-	<property name="cam_op" value="0.0" />
-	<property name="cam_oy" value="0.0" />
+	<xacro:property name="cam_px" value="0.029" />
+	<xacro:property name="cam_py" value="-0.01" />
+	<xacro:property name="cam_pz" value="0.019" />
+	<xacro:property name="cam_or" value="0.0" />
+	<xacro:property name="cam_op" value="0.0" />
+	<xacro:property name="cam_oy" value="0.0" />
 	<!-- imu properties -->
-	<property name="imu_pos_X" value="0.1885"/>
-	<property name="imu_pos_Y" value="0.0"/>
-	<property name="imu_pos_Z" value="0.108"/>
-	<property name="imu_or_R" value="0.0"/>
-	<property name="imu_or_P" value="0.0"/>
-	<property name="imu_or_Y" value="${-PI / 2}"/>
+	<xacro:property name="imu_pos_X" value="0.1885"/>
+	<xacro:property name="imu_pos_Y" value="0.0"/>
+	<xacro:property name="imu_pos_Z" value="0.108"/>
+	<xacro:property name="imu_or_R" value="0.0"/>
+	<xacro:property name="imu_or_P" value="0.0"/>
+	<xacro:property name="imu_or_Y" value="${-PI / 2}"/>
 </robot>

File: src/canyonero_description/urdf/sensors/canyonero_imu.urdf.xacro (robot description, xacro)
@@ -7,6 +7,6 @@
 <robot xmlns:xacro="http://ros.org/wiki/xacro">
   <xacro:macro name="imu_sensor" params="parent">
-    <joint name="$imu_joint" type="fixed">
-      <origin xyz="${imu_pos_X} ${imu_pos_Y} ${imu_pos_Z}" rpy = "${imu_or_R} ${imu_or_P} ${imu_or_Y}"/>
+    <joint name="imu_joint" type="fixed">
+      <origin xyz = "${imu_pos_X} ${imu_pos_Y} ${imu_pos_Z}" rpy = "${imu_or_R} ${imu_or_P} ${imu_or_Y}"/>
       <parent link="${parent}"/>
       <child link="imu_link"/>
@@ -20,4 +20,10 @@
         <material name="Red"/>
       </visual>
+      <collision>
+        <origin xyz="0.0 0.0 0.0" rpy="0 0 0"/>
+        <geometry>
+          <box size="0.27 0.40 0.5"/>
+        </geometry>
+      </collision>
       <inertial>
         <mass value="0.01"/>

File: src/canyonero_description/urdf/wheels/canyonero_wheel.urdf.xacro (robot description, xacro)
@@ -51,5 +51,5 @@
 				<kd value="1.0" />
 				<fdir1 value="1 0 0"/>
-				<material>Gazebo/Black</material>
+				<material value="Gazebo/Black"/>
 			</gazebo>
   	</xacro:macro>

File: src/canyonero_gazebo/urdf/canyonero.gazebo.xacro (robot description, xacro)
@@ -6,5 +6,6 @@
 -->
 <robot xmlns:xacro="http://ros.org/wiki/xacro">
-  <xacro:include filename="$(find canyonero_gazebo)/urdf/canyonero_sensors_gazebo.urdf.xacro"/>
+  <xacro:include filename="$(find canyonero_gazebo)/urdf/sensors/kinect.gazebo.xacro"/>
+  <xacro:include filename="$(find canyonero_gazebo)/urdf/sensors/imu.gazebo.xacro"/>
   <xacro:macro name="canyonero_robot_gazebo">
     <!-- Gazebo plugin for ROS Control -->
@@ -14,5 +15,10 @@
       </plugin>
     </gazebo>
-    <!--xacro:canyonero_sensors_gazebo/-->
+    <!-- Gazebo plugin for Kinect IR sensor -->
+    <xacro:kinect_ir_sensor link_name="camera_link" frame_name="camera_depth_frame" camera_name="kinect"/>
+    <!-- Gazebo plugin for Kinect RGB sensor -->
+    <xacro:kinect_rgb_sensor link_name="camera_link" frame_name="camera_rgb_frame" camera_name="kinect"/>
+    <!-- Gazebo plugin for IMU sensor -->
+    <xacro:imu_sensor_gazebo link_name="imu_link" imu_topic="imu_data" update_rate="100.0"/>
   </xacro:macro>
 </robot>
