Commit message: Debugging the messaging between ROS and Arduino.

File: canyonero_description/urdf/canyonero.urdf.xacro (robot description, xacro)
@@ -6,6 +6,13 @@
 -->
 <robot xmlns:xacro="http://ros.org/wiki/xacro" name="canyonero">
+	<xacro:include filename="$(find canyonero_description)/urdf/canyonero_properties.urdf.xacro"/>"
 	<xacro:include filename="$(find canyonero_description)/urdf/canyonero_base.urdf.xacro"/>
+	<xacro:include filename="$(find canyonero_description)/urdf/sensors/canyonero_kinect.urdf.xacro"/>
+	<xacro:include filename="$(find canyonero_description)/urdf/sensors/canyonero_imu.urdf.xacro"/>
 	<!-- Base -->
 	<xacro:base name="base"/>
+	<!-- 3D sensor -->
+	<xacro:sensor_kinect parent="base_link"/>
+	<!-- IMU -->
+	<xacro:imu_sensor parent="base_link" update_rate="100.0"/>
 </robot>

File: canyonero_description/urdf/canyonero_base.urdf.xacro (robot description, xacro)
@@ -6,6 +6,5 @@
 -->
 <robot xmlns:xacro="http://ros.org/wiki/xacro">
-	<xacro:include filename="$(find canyonero_description)/urdf/canyonero_wheel.urdf.xacro"/>
-	<property name="pos_Z2"       value="1.67"/>
+	<xacro:include filename="$(find canyonero_description)/urdf/wheels/canyonero_wheel.urdf.xacro"/>
 	<xacro:macro name= "base" params = "name">
 	<!-- BASE-FOOTPRINT -->
@@ -15,5 +14,5 @@
 			<parent link = "${name}_footprint"/>
 			<child link = "${name}_link"/>
-			<origin xyz = "0 0 ${pos_Z2}" rpy = "0 0 0"/>
+			<origin xyz = "0 0 ${rob_pos_Z}" rpy = "0 0 0"/>
 		</joint>
 		<!-- BASE-LINK -->
@@ -25,31 +24,33 @@
 					<mesh filename = "package://canyonero_description/meshes/canyonero_plates.stl"/>
 				</geometry>
-				<material name = "cambot/red">
-					<color rgba = "1.0 0.0 0.0 1"/>
-				</material>
+				<material name = "Red"/>
 			</visual>
-			<!--collision>
+			<collision>
 	      		<origin xyz = "0 0 0" rpy = "0 0 0"/>
 	      		<geometry>
 	        		<mesh filename = "package://canyonero_description/meshes/canyonero_plates_collision.stl"/>
 	      		</geometry>
-	    	</collision-->
+	    	</collision>
 			<inertial>
-	      		<origin rpy = "0 0 0" xyz = "174.84e-3 117.51e-3 -218.86e-3"/>
-	      		<mass value = "15.23"/>
-	      		<!-- inertia at cm or origin?-->
-	      		<inertia ixx = "0.016258"
-	               		 ixy = "0.000432"
-	               		 ixz="-0.000049"
-	               		 iyy="0.019275"
-	               		 iyz="0.000048"
-	               		 izz="0.016834"/>
+	      		<origin xyz="0.023661 -0.000069 -0.036285" rpy="0 0 0" />
+	      		<mass value = "10"/>
+	      		<inertia ixx="0.5284" ixy="-0.0003498" ixz="0.001138"
+	               		 iyy="0.5262" iyz="0.02108"
+	               		 izz="0.9556"/>
 	    	</inertial>
+				<gazebo reference="${name}_link">
+      		<material>Gazebo/Red</material>
+    		</gazebo>
 		</link>
 		<!-- Wheels -->
-	    <xacro:wheel sideY = "frontal" sideX = "left" positionY = "1.0" positionX = "1.0" reflect = "-1.0" parent = "${name}"/>
-	    <xacro:wheel sideY = "frontal" sideX = "right" positionY = "1.0" positionX = "-1.0" reflect = "1.0" parent = "${name}"/>
-	    <xacro:wheel sideY = "back" sideX = "left" positionY = "-1.0" positionX = "1.0" reflect = "-1.0" parent = "${name}"/>
-	    <xacro:wheel sideY = "back" sideX = "right" positionY = "-1.0" positionX = "-1.0" reflect = "1.0" parent = "${name}"/>
+	    <xacro:wheel sideX = "frontal" sideY = "left" positionX = "1.0" positionY = "1.0" reflect = "-1.0" parent = "${name}"/>
+	    <xacro:wheel sideX = "frontal" sideY = "right" positionX = "1.0" positionY = "-1.0" reflect = "1.0" parent = "${name}"/>
+	    <xacro:wheel sideX = "back" sideY = "left" positionX = "-1.0" positionY = "1.0" reflect = "-1.0" parent = "${name}"/>
+	    <xacro:wheel sideX = "back" sideY = "right" positionX = "-1.0" positionY = "-1.0" reflect = "1.0" parent = "${name}"/>
+			<gazebo>
+				<plugin name="gazebo_ros_control" filename="libgazebo_ros_control.so">
+				<robotNamespace>canyonero</robotNamespace>
+				</plugin>
+			</gazebo>
 	</xacro:macro>
 </robot>

File: canyonero_description/urdf/canyonero_wheel.urdf.xacro (robot description, xacro)
@@ -5,37 +5,35 @@
   Creative Commons, 444 Castro Street, Suite 900, Mountain View, California, 94041, USA.
 -->
-<robot xmlns:xacro="http://ros.org/wiki/xacro">
-	<property name="pos_X"       value="1.62"/>
-	<property name="pos_Y"       value="1.65"/>
-	<!--property name="pos_Z"       value="-0.68"/-->
+<robot xmlns:xacro = "http://ros.org/wiki/xacro">
 	<xacro:macro name="wheel" params="sideY sideX positionY positionX reflect parent">
 	    <link name="${sideY}_${sideX}_wheel_link">
 	    	<visual>
-	        	<origin xyz = "0 0 0" rpy = "0 -1.57 0"/>
+	        	<origin xyz = "0 0 0" rpy = "0 ${-PI / 2} 0"/>
 	        	<geometry>
 	          		<mesh filename="package://canyonero_description/meshes/canyonero_wheel.stl"/>
 	        	</geometry>
-	        	<material name = "cambot/black">
-					<color rgba = "0.0 0.0 0.0 1.0"/>
-				</material>
+	        	<material name = "Black"/>
 	      	</visual>
-		    <!--inertial>
-		    	<origin xyz="1.62*${positionX} 1.65*${positionY} -0.68" rpy="1.57*${reflect} 0 0"/>
-		        <mass value="1.82362"/>
-		        <inertia ixx="0.00499743171" ixy="${ 0.00000004464 * reflect}" ixz="-0.00000002245"
-		                 iyy="0.00499741733" iyz="${-0.00000000164 * reflect}"
-		                 izz="0.00839239692"/>
-		    </inertial-->
-	      	<!--collision>
+		    <inertial>
+		    	<origin xyz="0.1026 0.0 0.0" rpy="0 0 0"/>
+		        <mass value="1.419"/>
+		        <inertia ixx="0.0165" ixy="0.0" ixz="0.0"
+		                 iyy="0.0106" iyz="0.0"
+		                 izz="0.0106"/>
+		    </inertial>
+	      	<collision>
 	        	<origin xyz="0 0 0" rpy="0 0 0"/>
 	        	<geometry>
-	          		<mesh filename = "package://canyonero_description/meshes/canyonero_wheel.stl"/>
+	          		<mesh filename = "package://canyonero_description/meshes/canyonero_wheel_collision.stl"/>
 	        	</geometry>
-	      	</collision-->
+	      	</collision>
+	      	<gazebo reference="${sideY}_${sideX}_wheel_link">
+      			<material>Gazebo/Black</material>
+    		</gazebo>
 	    </link>
 	    <joint name="${sideY}_${sideX}_wheel_joint" type="continuous">
 	    	<parent link="${parent}_link"/>
 	      	<child link="${sideY}_${sideX}_wheel_link"/>
-	      	<origin xyz="${pos_X}*${positionX} ${pos_Y}*${positionY} ${pos_Z}" rpy="1.57*${reflect} 0 0"/>
+	      	<origin xyz="${wheel_pos_X * positionX} ${wheel_pos_Y * positionY} ${-wheel_pos_Z}" rpy="${(PI / 2) * reflect} 0 0"/>
 	      	<axis xyz="0 0 1"/>
 	    </joint>

Commit message: updating canyonero_gazebo and canyonero_description at the roscontrol branch

File: canyonero_description/urdf/canyonero.urdf.xacro (robot description, xacro)
@@ -6,13 +6,16 @@
 -->
 <robot xmlns:xacro="http://ros.org/wiki/xacro" name="canyonero">
-	<xacro:include filename="$(find canyonero_description)/urdf/canyonero_properties.urdf.xacro"/>"
-	<xacro:include filename="$(find canyonero_description)/urdf/canyonero_base.urdf.xacro"/>
-	<xacro:include filename="$(find canyonero_description)/urdf/sensors/canyonero_kinect.urdf.xacro"/>
-	<xacro:include filename="$(find canyonero_description)/urdf/sensors/canyonero_imu.urdf.xacro"/>
-	<!-- Base -->
-	<xacro:base name="base"/>
-	<!-- 3D sensor -->
-	<xacro:sensor_kinect parent="base_link"/>
-	<!-- IMU -->
-	<xacro:imu_sensor parent="base_link" update_rate="100.0"/>
+		<xacro:include filename="$(find canyonero_description)/urdf/canyonero_properties.urdf.xacro"/>"
+		<xacro:include filename="$(find canyonero_description)/urdf/canyonero_base.urdf.xacro"/>
+		<xacro:include filename="$(find canyonero_description)/urdf/sensors/canyonero_kinect.urdf.xacro"/>
+		<xacro:include filename="$(find canyonero_description)/urdf/sensors/canyonero_imu.urdf.xacro"/>
+		<xacro:include filename="$(find canyonero_gazebo)/urdf/canyonero.gazebo.xacro"/>
+		<!-- Base -->
+		<xacro:wheeled_base name="base"/>
+		<!-- 3D sensor -->
+		<xacro:sensor_kinect parent="base_link"/>
+		<!-- IMU -->
+		<xacro:imu_sensor parent="base_link"/>
+		<!-- Gazebo -->
+		<xacro:canyonero_robot_gazebo/>
 </robot>

File: canyonero_description/urdf/canyonero_base.urdf.xacro (robot description, xacro)
@@ -7,5 +7,5 @@
 <robot xmlns:xacro="http://ros.org/wiki/xacro">
 	<xacro:include filename="$(find canyonero_description)/urdf/wheels/canyonero_wheel.urdf.xacro"/>
-	<xacro:macro name= "base" params = "name">
+	<xacro:macro name= "wheeled_base" params = "name">
 	<!-- BASE-FOOTPRINT -->
 		<!-- base_footprint is a fictitious link(frame) that is on the ground right below base_link origin, navigation stack depends on this frame -->
@@ -24,5 +24,5 @@
 					<mesh filename = "package://canyonero_description/meshes/canyonero_plates.stl"/>
 				</geometry>
-				<material name = "Red"/>
+				<material name="Red"/>
 			</visual>
 			<collision>
@@ -34,23 +34,18 @@
 			<inertial>
 	      		<origin xyz="0.023661 -0.000069 -0.036285" rpy="0 0 0" />
-	      		<mass value = "10"/>
-	      		<inertia ixx="0.5284" ixy="-0.0003498" ixz="0.001138"
-	               		 iyy="0.5262" iyz="0.02108"
-	               		 izz="0.9556"/>
-	    	</inertial>
-				<gazebo reference="${name}_link">
-      		<material>Gazebo/Red</material>
-    		</gazebo>
+	      		<mass value="10"/>
+	      		<inertia ixx="0.27658267" ixy="0.0" ixz="-0.02663389"
+	               		 iyy="0.38926449" iyz="0.0"
+	               		 izz="0.57775046"/>
+	    </inertial>
 		</link>
+		<gazebo reference="${name}_link">
+      <material value="Gazebo/Red"/>
+    </gazebo>
 		<!-- Wheels -->
-	    <xacro:wheel sideX = "frontal" sideY = "left" positionX = "1.0" positionY = "1.0" reflect = "-1.0" parent = "${name}"/>
-	    <xacro:wheel sideX = "frontal" sideY = "right" positionX = "1.0" positionY = "-1.0" reflect = "1.0" parent = "${name}"/>
-	    <xacro:wheel sideX = "back" sideY = "left" positionX = "-1.0" positionY = "1.0" reflect = "-1.0" parent = "${name}"/>
-	    <xacro:wheel sideX = "back" sideY = "right" positionX = "-1.0" positionY = "-1.0" reflect = "1.0" parent = "${name}"/>
-			<gazebo>
-				<plugin name="gazebo_ros_control" filename="libgazebo_ros_control.so">
-				<robotNamespace>canyonero</robotNamespace>
-				</plugin>
-			</gazebo>
+	    <xacro:wheel sideX = "frontal" sideY = "left" positionX = "1.0" positionY = "1.0" reflect = "-1.0" parent = "${name}" torque="${wheel_torque}" velocity="${wheel_velocity}" radius="${wheel_radius}" />
+	    <xacro:wheel sideX = "frontal" sideY = "right" positionX = "1.0" positionY = "-1.0" reflect = "1.0" parent = "${name}" torque="${wheel_torque}" velocity="${wheel_velocity}" radius="${wheel_radius}"/>
+	    <xacro:wheel sideX = "back" sideY = "left" positionX = "-1.0" positionY = "1.0" reflect = "-1.0" parent = "${name}" torque="${wheel_torque}" velocity="${wheel_velocity}" radius="${wheel_radius}"/>
+	    <xacro:wheel sideX = "back" sideY = "right" positionX = "-1.0" positionY = "-1.0" reflect = "1.0" parent = "${name}" torque="${wheel_torque}" velocity="${wheel_velocity}" radius="${wheel_radius}"/>
 	</xacro:macro>
 </robot>

File: canyonero_description/urdf/canyonero_properties.urdf.xacro (robot description, xacro)
@@ -19,9 +19,12 @@
 	<!-- base properties -->
 	<!-- robot's elevation from the ground -->
-	<property name = "rob_pos_Z"	value = "0.167"/>
+	<xacro:property name="rob_pos_Z" value="0.167"/>
 	<!-- wheel properties -->
-	<property name = "wheel_pos_X"      value = "0.162"/>
-	<property name = "wheel_pos_Y"      value = "0.165"/>
-	<property name = "wheel_pos_Z"			value = "0.068"/>
+	<xacro:property name="wheel_pos_X" value="0.162"/>
+	<xacro:property name="wheel_pos_Y" value="0.165"/>
+	<xacro:property name="wheel_pos_Z" value="0.068"/>
+	<xacro:property name="wheel_torque" value="1.0"/>
+	<xacro:property name="wheel_velocity" value="1.0"/>
+	<xacro:property name="wheel_radius" value="0.20"/>
 	<!-- kinect properties -->
 	<!-- kinect position at the robot -->

File: canyonero_description/urdf/sensors/canyonero_imu.urdf.xacro (robot description, xacro)
@@ -6,6 +6,6 @@
 -->
 <robot xmlns:xacro="http://ros.org/wiki/xacro">
-  <xacro:macro name="imu_sensor" params="parent update_rate">
-    <joint name="$imu_joint" type="fixed">
+  <xacro:macro name="imu_sensor" params="parent">
+    <joint name="imu_joint" type="fixed">
       <origin xyz = "${imu_pos_X} ${imu_pos_Y} ${imu_pos_Z}" rpy = "${imu_or_R} ${imu_or_P} ${imu_or_Y}"/>
       <parent link="${parent}"/>
@@ -18,6 +18,12 @@
           <mesh filename = "package://canyonero_description/meshes/9dof_razor_imu.stl" scale="0.1 0.1 0.1"/>
         </geometry>
-        <material name = "Red"/>
+        <material name="Red"/>
       </visual>
+      <collision>
+        <origin xyz="0.0 0.0 0.0" rpy="0 0 0"/>
+        <geometry>
+          <box size="0.27 0.40 0.5"/>
+        </geometry>
+      </collision>
       <inertial>
         <mass value="0.01"/>
@@ -26,28 +32,4 @@
       </inertial>
     </link>
-    <gazebo reference="imu_link">
-      <sensor name="imu_sensor" type="imu">
-        <always_on>1</always_on>
-        <update_rate>100.0</update_rate>
-        <imu>
-          <noise>
-            <type>gaussian</type>
-            <rate>
-              <mean>0.0</mean>
-              <stddev>2e-4</stddev>
-              <bias_mean>0.0000075</bias_mean>
-              <bias_stddev>0.0000008</bias_stddev>
-            </rate>
-            <accel>
-              <mean>0.0</mean>
-              <stddev>1.7e-2</stddev>
-              <bias_mean>0.1</bias_mean>
-              <bias_stddev>0.001</bias_stddev>
-            </accel>
-          </noise>
-        </imu>
-      </sensor>
-      <material>Gazebo/Red</material>
-    </gazebo>
   </xacro:macro>
 </robot>

File: canyonero_description/urdf/wheels/canyonero_wheel.urdf.xacro (robot description, xacro)
@@ -6,5 +6,5 @@
 -->
 <robot xmlns:xacro = "http://ros.org/wiki/xacro">
-	<xacro:macro name="wheel" params="sideY sideX positionY positionX reflect parent">
+	<xacro:macro name="wheel" params="sideY sideX positionY positionX reflect parent torque velocity radius">
 	    <link name="${sideY}_${sideX}_wheel_link">
 	    	<visual>
@@ -13,22 +13,19 @@
 	          		<mesh filename="package://canyonero_description/meshes/canyonero_wheel.stl"/>
 	        	</geometry>
-	        	<material name = "Black"/>
+	        	<material name="Black"/>
 	      	</visual>
 		    <inertial>
 		    	<origin xyz="0.0 0.0 0.102638" rpy="0 0 0"/>
 		        <mass value="1.419"/>
-		        <inertia ixx="0.01101" ixy="0.0000238" ixz="0.00000223198"
-				        		 iyy="0.01104" iyz="${-0.00000012456 * reflect}"
-				             izz="0.003326"/>
+		        <inertia ixx="0.00305" ixy="0.0" ixz="0.0"
+				        		 iyy="0.00305" iyz="0.0"
+				             izz="0.00512"/>
 		    </inertial>
 	      	<collision>
 	        	<origin xyz="0 0 0" rpy="0 ${-PI / 2} 0"/>
 	        	<geometry>
-	          		<mesh filename = "package://canyonero_description/meshes/canyonero_wheel_collision.stl"/>
+	          		<mesh filename="package://canyonero_description/meshes/canyonero_wheel_collision.stl"/>
 	        	</geometry>
 	      	</collision>
-	      	<gazebo reference="${sideY}_${sideX}_wheel_link">
-      			<material>Gazebo/Black</material>
-    		</gazebo>
 	    </link>
 	    <joint name="${sideY}_${sideX}_wheel_joint" type="continuous">
@@ -37,15 +34,23 @@
 	      	<origin xyz="${wheel_pos_X * positionX} ${wheel_pos_Y * positionY} ${-wheel_pos_Z}" rpy="${(PI / 2) * reflect} 0 0"/>
 	      	<axis xyz="0 0 1"/>
+					<limit effort="${torque}" velocity="${velocity / radius}"/>
 	    </joint>
 			<transmission name="simple_trans">
 			  <type>transmission_interface/SimpleTransmission</type>
 			  <joint name="${sideY}_${sideX}_wheel_joint">
-					<hardwareInterface>EffortJointInterface</hardwareInterface>
+					<hardwareInterface>VelocityJointInterface</hardwareInterface>
 			  </joint>
 			  <actuator name="DC_motor">
 					<mechanicalReduction>1</mechanicalReduction>
-					<hardwareInterface>EffortJointInterface</hardwareInterface>
 			  </actuator>
 			</transmission>
+			<gazebo reference="${sideY}_${sideX}_wheel_link">
+				<mu1 value="1.0"/>
+				<mu2 value="1.0"/>
+				<kp value="10000000.0" />
+				<kd value="1.0" />
+				<fdir1 value="1 0 0"/>
+				<material value="Gazebo/Black"/>
+			</gazebo>
   	</xacro:macro>
 </robot>
