Commit message: Preparing sim.launch for the 5 different practices

File: canyonero_description/urdf/canyonero_properties.urdf.xacro (robot description, xacro)
@@ -25,5 +25,5 @@
 	<xacro:property name="wheel_pos_Z" value="0.068"/>
 	<xacro:property name="wheel_torque" value="1.0"/>
-	<xacro:property name="wheel_velocity" value="1.0"/>
+	<xacro:property name="wheel_velocity" value="3.0"/>
 	<xacro:property name="wheel_radius" value="0.20"/>
 	<!-- kinect properties -->

File: canyonero_description/urdf/wheels/canyonero_wheel.urdf.xacro (robot description, xacro)
@@ -46,9 +46,9 @@
 			</transmission>
 			<gazebo reference="wheel_${sideX}_${sideY}_link">
-				<mu1 value="1.0"/>
-				<mu2 value="1.0"/>
-				<kp value="10000000.0" />
-				<kd value="1.0" />
-				<fdir1 value="1 0 0"/>
+				<mu1 value="0.75"/>
+				<mu2 value="0.75"/>
+				<!--kp value="10000000.0" /-->
+				<!--kd value="1.0" /-->
+				<fdir1 value="0 0 0"/>
 				<material value="Gazebo/Black"/>
 			</gazebo>
