Commit message: It moves! (although it seems there is a problem with the axis...)

File: canyonero_description/urdf/canyonero_base.urdf.xacro (robot description, xacro)
@@ -44,8 +44,8 @@
     </gazebo>
 		<!-- Wheels -->
-	    <xacro:wheel sideX = "frontal" sideY = "left" positionX = "1.0" positionY = "1.0" reflect = "-1.0" parent = "${name}" torque="${wheel_torque}" velocity="${wheel_velocity}" radius="${wheel_radius}" />
-	    <xacro:wheel sideX = "frontal" sideY = "right" positionX = "1.0" positionY = "-1.0" reflect = "1.0" parent = "${name}" torque="${wheel_torque}" velocity="${wheel_velocity}" radius="${wheel_radius}"/>
-	    <xacro:wheel sideX = "back" sideY = "left" positionX = "-1.0" positionY = "1.0" reflect = "-1.0" parent = "${name}" torque="${wheel_torque}" velocity="${wheel_velocity}" radius="${wheel_radius}"/>
-	    <xacro:wheel sideX = "back" sideY = "right" positionX = "-1.0" positionY = "-1.0" reflect = "1.0" parent = "${name}" torque="${wheel_torque}" velocity="${wheel_velocity}" radius="${wheel_radius}"/>
+	    <xacro:wheel sideX = "front" sideY = "left" positionX = "1.0" positionY = "1.0" reflect = "-1.0" parent = "${name}" torque="${wheel_torque}" velocity="${wheel_velocity}" radius="${wheel_radius}" />
+	    <xacro:wheel sideX = "front" sideY = "right" positionX = "1.0" positionY = "-1.0" reflect = "1.0" parent = "${name}" torque="${wheel_torque}" velocity="${wheel_velocity}" radius="${wheel_radius}"/>
+	    <xacro:wheel sideX = "rear" sideY = "left" positionX = "-1.0" positionY = "1.0" reflect = "-1.0" parent = "${name}" torque="${wheel_torque}" velocity="${wheel_velocity}" radius="${wheel_radius}"/>
+	    <xacro:wheel sideX = "rear" sideY = "right" positionX = "-1.0" positionY = "-1.0" reflect = "1.0" parent = "${name}" torque="${wheel_torque}" velocity="${wheel_velocity}" radius="${wheel_radius}"/>
 	</xacro:macro>
 </robot>

File: canyonero_description/urdf/wheels/canyonero_wheel.urdf.xacro (robot description, xacro)
@@ -7,5 +7,5 @@
 <robot xmlns:xacro = "http://ros.org/wiki/xacro">
 	<xacro:macro name="wheel" params="sideY sideX positionY positionX reflect parent torque velocity radius">
-	    <link name="${sideY}_${sideX}_wheel_link">
+	    <link name="wheel_${sideX}_${sideY}_link">
 	    	<visual>
 	        	<origin xyz = "0 0 0" rpy = "0 ${-PI / 2} 0"/>
@@ -29,7 +29,7 @@
 	      	</collision>
 	    </link>
-	    <joint name="${sideY}_${sideX}_wheel_joint" type="continuous">
+	    <joint name="wheel_${sideX}_${sideY}_joint" type="continuous">
 	    	<parent link="${parent}_link"/>
-	      	<child link="${sideY}_${sideX}_wheel_link"/>
+	      	<child link="wheel_${sideX}_${sideY}_link"/>
 	      	<origin xyz="${wheel_pos_X * positionX} ${wheel_pos_Y * positionY} ${-wheel_pos_Z}" rpy="${(PI / 2) * reflect} 0 0"/>
 	      	<axis xyz="0 0 1"/>
@@ -38,5 +38,5 @@
 			<transmission name="simple_trans">
 			  <type>transmission_interface/SimpleTransmission</type>
-			  <joint name="${sideY}_${sideX}_wheel_joint">
+			  <joint name="wheel_${sideX}_${sideY}_joint">
 					<hardwareInterface>VelocityJointInterface</hardwareInterface>
 			  </joint>
@@ -45,5 +45,5 @@
 			  </actuator>
 			</transmission>
-			<gazebo reference="${sideY}_${sideX}_wheel_link">
+			<gazebo reference="wheel_${sideX}_${sideY}_link">
 				<mu1 value="1.0"/>
 				<mu2 value="1.0"/>

Commit message: Updating Canyonero_Gazebo

File: canyonero_description/urdf/canyonero_base.urdf.xacro (robot description, xacro)
@@ -44,8 +44,8 @@
     </gazebo>
 		<!-- Wheels -->
-	    <xacro:wheel sideX = "front" sideY = "left" positionX = "1.0" positionY = "1.0" reflect = "-1.0" parent = "${name}" torque="${wheel_torque}" velocity="${wheel_velocity}" radius="${wheel_radius}" />
-	    <xacro:wheel sideX = "front" sideY = "right" positionX = "1.0" positionY = "-1.0" reflect = "1.0" parent = "${name}" torque="${wheel_torque}" velocity="${wheel_velocity}" radius="${wheel_radius}"/>
-	    <xacro:wheel sideX = "rear" sideY = "left" positionX = "-1.0" positionY = "1.0" reflect = "-1.0" parent = "${name}" torque="${wheel_torque}" velocity="${wheel_velocity}" radius="${wheel_radius}"/>
-	    <xacro:wheel sideX = "rear" sideY = "right" positionX = "-1.0" positionY = "-1.0" reflect = "1.0" parent = "${name}" torque="${wheel_torque}" velocity="${wheel_velocity}" radius="${wheel_radius}"/>
+	    <xacro:wheel sideX = "front" sideY = "left" positionX = "1.0" positionY = "1.0" reflect = "-1.0" axis_z = "1" parent = "${name}" torque="${wheel_torque}" velocity="${wheel_velocity}" radius="${wheel_radius}" />
+	    <xacro:wheel sideX = "front" sideY = "right" positionX = "1.0" positionY = "-1.0" reflect = "1.0" axis_z = "-1" parent = "${name}" torque="${wheel_torque}" velocity="${wheel_velocity}" radius="${wheel_radius}"/>
+	    <xacro:wheel sideX = "rear" sideY = "left" positionX = "-1.0" positionY = "1.0" reflect = "-1.0" axis_z = "1" parent = "${name}" torque="${wheel_torque}" velocity="${wheel_velocity}" radius="${wheel_radius}"/>
+	    <xacro:wheel sideX = "rear" sideY = "right" positionX = "-1.0" positionY = "-1.0" reflect = "1.0" axis_z = "-1" parent = "${name}" torque="${wheel_torque}" velocity="${wheel_velocity}" radius="${wheel_radius}"/>
 	</xacro:macro>
 </robot>

File: canyonero_description/urdf/wheels/canyonero_wheel.urdf.xacro (robot description, xacro)
@@ -6,5 +6,5 @@
 -->
 <robot xmlns:xacro = "http://ros.org/wiki/xacro">
-	<xacro:macro name="wheel" params="sideY sideX positionY positionX reflect parent torque velocity radius">
+	<xacro:macro name="wheel" params="sideY sideX positionY positionX reflect axis_z parent torque velocity radius">
 	    <link name="wheel_${sideX}_${sideY}_link">
 	    	<visual>
@@ -33,6 +33,6 @@
 	      	<child link="wheel_${sideX}_${sideY}_link"/>
 	      	<origin xyz="${wheel_pos_X * positionX} ${wheel_pos_Y * positionY} ${-wheel_pos_Z}" rpy="${(PI / 2) * reflect} 0 0"/>
-	      	<axis xyz="0 0 1"/>
-					<limit effort="${torque}" velocity="${velocity / radius}"/>
+	      	<axis xyz="0 0 ${axis_z}"/>
+			<limit effort="${torque}" velocity="${velocity / radius}"/>
 	    </joint>
 			<transmission name="simple_trans">
